File: HW/Untitled/Untitled.kicad_sch (KiCad schematic)
At the start: 0 parts

Commit message: Solid version of FW with screen flipping capabilities and furhter improved UI along with initial .sch and .brd files for the peripheral circuit
Parts:
- added J1: Sparkfun, symbol Connector_Generic:Conn_01x15
- added Q1, Q2: 2N7000, Package_TO_SOT_THT:TO-92_Inline, symbol Transistor_FET:2N7000
Connections:
- new net: J1.8 (Pin_8), Q2.3 (D)
- new net: J1.Vcc (Pin_1), Q1.3 (D)
- new net +3V3: Q1.1 (S), Q2.1 (S)
- new net D0: Q1.2 (G)
- new net D18: Q2.2 (G)
