File: HW/Untitled/textmachine_peripheral_circuit.kicad_sch (KiCad schematic)
At the start: 32 parts, among them J1 Sparkfun, J2 Sparkfun, Q1 2N7000, Q2 2N7000, Q3 2N7000, Q4 2N7000, X1 332-06, X2 332-06

Commit message: UI Improvements
Parts:
- added C2: 0.1uF, SparkFun_Buck_Regulator_AP63357DV-7_Buck5V:0402-TIGHT, symbol SparkFun_Buck_Regulator_AP63357DV-7_Buck5V-eagle-import:0.1UF-0402T-16V-10%
- added C2: 47pF, SparkFun_Buck_Regulator_AP63357DV-7_Buck5V:0402-TIGHT, symbol SparkFun_Buck_Regulator_AP63357DV-7_Buck5V-eagle-import:47PF-0402_TIGHT-25V-5%-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
- added C4 (x2): 22uF, SparkFun_Buck_Regulator_AP63357DV-7_Buck5V:0805, symbol SparkFun_Buck_Regulator_AP63357DV-7_Buck5V-eagle-import:22UF-0805-16V-20%
- added C5, C6: 4.7uF, SparkFun_Buck_Regulator_AP63357DV-7_Buck5V:0805, symbol SparkFun_Buck_Regulator_AP63357DV-7_Buck5V-eagle-import:4.7UF-0805-50V-(10%)
- added L1: 6.8UH, SparkFun_Buck_Regulator_AP63357DV-7_Buck5V:07A7_6U8H, symbol SparkFun_Buck_Regulator_AP63357DV-7_Buck5V-eagle-import:6.8UH
- added R3: 220K, SparkFun_Buck_Regulator_AP63357DV-7_Buck5V:0402-TIGHT, symbol SparkFun_Buck_Regulator_AP63357DV-7_Buck5V-eagle-import:220KOHM-0402T-1/16W-1%
- added R3: 93.1k, SparkFun_Buck_Regulator_AP63357DV-7_Buck5V:0402-TIGHT, symbol SparkFun_Buck_Regulator_AP63357DV-7_Buck5V-eagle-import:93.1KOHM-0402-1/16W-1%(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
- added R4: 22k, SparkFun_Buck_Regulator_AP63357DV-7_Buck5V:0402-TIGHT, symbol SparkFun_Buck_Regulator_AP63357DV-7_Buck5V-eagle-import:22KOHM-0402_TIGHT-1/10W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
- added R4: 41.2K, SparkFun_Buck_Regulator_AP63357DV-7_Buck5V:0402-TIGHT, symbol SparkFun_Buck_Regulator_AP63357DV-7_Buck5V-eagle-import:41.2KOHM-0402-1/16W-1%(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
- added S4: EVQ-P7L01P, power_circuit:SW_EVQ-P7L01P, symbol power_circuit-eagle-import:EVQ-P7L01P
- added U1: BQ25173DSG, Package_SON:WSON-8-1EP_2x2mm_P0.5mm_EP0.9x1.6mm, symbol Battery_Management:BQ25173DSG
- added U2: AP63357, SparkFun_Buck_Regulator_AP63357DV-7_Buck5V:V-DFN3020-13, symbol SparkFun_Buck_Regulator_AP63357DV-7_Buck5V-eagle-import:AP63357
- C1: value C5/3 -> 1F
- D2: OC_NEWARK unknown -> (none)
Connections:
- net GND2 is gone; now on net GND: BUCK_CRG0.4 (S), BUCK_CRG1.4 (S), C1.2, C3.2, R1.1, R2.1
- net GND: now also C4.2, C4.2, C5.2, C6.2, R4.1, R4.1, U1.4 (GND), U1.9 (GND), U2.P$4 (COMP), U2.P$8 (GND)
- net VBAT: no longer BUCK_CRG1.2 (S), S3.2_1 (2), S3.2_2 (2)
- net Vbat: now reaches C1.1, S3.1_1 (1), S3.1_2 (1)
- net Vbat: now also S4.2_1 (2), S4.2_2 (2); no longer R2.2
- net Vcc (screen): now reaches Q1.2 (G), S5.1_1 (1), S5.1_2 (1)
- net Vcc (screen): now also Q1.3 (D)
- net at Q2.3 (D): no longer J1.8 (Pin_8)
- net at J1.Vcc (Pin_1): no longer Q1.3 (D)
- new net: C2.1, U2.P$6 (BST)
- new net: C2.2, L1.P$1 (1), U2.P$7 (SW), U2.P$9 (SW)
- new net: C2.2, R3.1, R4.2, U2.P$3 (FB)
- new net: R2.2, S4.1_1 (1), S4.1_2 (1)
- new net: S3.2_1 (2), S3.2_2 (2), U1.8 (OUT)
- new net 5V: BUCK_CRG1.2 (S), C2.1, C4.1, C4.1, L1.P$2 (2), R3.2, U1.1 (IN)
- new net EN: R3.1, R4.2, U2.P$2 (EN)
- new net VIN: C5.1, C6.1, R3.2, U2.P$1 (VIN)
Other:
- note added: "5V switching buck regulator"
- note added: "TM : ON/OFF"
- note added: "UVLO Hi: 5.6V UVLO Lo: 5.18V See Datasheet pg 15 Eq. 2+3 For calculating R3/R4"
- note removed: "V_bat"
- moved on the sheet: A1, BUCK_CRG1A, BUCK_CRG1B, BUCK_CRG1C, BUCK_CRG1D, C1, D10, D2, D4, D5, D6, D8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

Commit message: Ported arduino to platformIO and 3 phase dynamo seciton of peripheral board done
Parts:
- removed C2: 0.1uF, SparkFun_Buck_Regulator_AP63357DV-7_Buck5V:0402-TIGHT, symbol SparkFun_Buck_Regulator_AP63357DV-7_Buck5V-eagle-import:0.1UF-0402T-16V-10%
- removed C2: 47pF, SparkFun_Buck_Regulator_AP63357DV-7_Buck5V:0402-TIGHT, symbol SparkFun_Buck_Regulator_AP63357DV-7_Buck5V-eagle-import:47PF-0402_TIGHT-25V-5%-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
- removed C4 (x2): 22uF, SparkFun_Buck_Regulator_AP63357DV-7_Buck5V:0805, symbol SparkFun_Buck_Regulator_AP63357DV-7_Buck5V-eagle-import:22UF-0805-16V-20%
- removed C5, C6: 4.7uF, SparkFun_Buck_Regulator_AP63357DV-7_Buck5V:0805, symbol SparkFun_Buck_Regulator_AP63357DV-7_Buck5V-eagle-import:4.7UF-0805-50V-(10%)
- removed L1: 6.8UH, SparkFun_Buck_Regulator_AP63357DV-7_Buck5V:07A7_6U8H, symbol SparkFun_Buck_Regulator_AP63357DV-7_Buck5V-eagle-import:6.8UH
- removed Q2: 2N7000, Package_TO_SOT_THT:TO-92_Inline, symbol Transistor_FET:2N7000
- removed R3: 220K, SparkFun_Buck_Regulator_AP63357DV-7_Buck5V:0402-TIGHT, symbol SparkFun_Buck_Regulator_AP63357DV-7_Buck5V-eagle-import:220KOHM-0402T-1/16W-1%
- removed R3: 93.1k, SparkFun_Buck_Regulator_AP63357DV-7_Buck5V:0402-TIGHT, symbol SparkFun_Buck_Regulator_AP63357DV-7_Buck5V-eagle-import:93.1KOHM-0402-1/16W-1%(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
- removed R4: 22k, SparkFun_Buck_Regulator_AP63357DV-7_Buck5V:0402-TIGHT, symbol SparkFun_Buck_Regulator_AP63357DV-7_Buck5V-eagle-import:22KOHM-0402_TIGHT-1/10W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
- removed R4: 41.2K, SparkFun_Buck_Regulator_AP63357DV-7_Buck5V:0402-TIGHT, symbol SparkFun_Buck_Regulator_AP63357DV-7_Buck5V-eagle-import:41.2KOHM-0402-1/16W-1%(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
- removed U1: BQ25173DSG, Package_SON:WSON-8-1EP_2x2mm_P0.5mm_EP0.9x1.6mm, symbol Battery_Management:BQ25173DSG
- removed U2: AP63357, SparkFun_Buck_Regulator_AP63357DV-7_Buck5V:V-DFN3020-13, symbol SparkFun_Buck_Regulator_AP63357DV-7_Buck5V-eagle-import:AP63357
- added Q2: Q_PMOS_GSD, symbol Transistor_FET:Q_PMOS_GSD
Connections:
- net D18: no longer A1.A3
- net GND: no longer BUCK_CRG0.4 (S), BUCK_CRG1.4 (S), C1.2, C3.2, R1.1, R2.1
- net at J1.8 (Pin_8): now also A1.A3
- net 5V: no longer names the net of BUCK_CRG1.2 (S)
- new net GND2: BUCK_CRG0.4 (S), BUCK_CRG1.4 (S), C1.2, C3.2, R1.1, R2.1
Other:
- note added: "brightness PWM (0-255)"
- note removed: "UVLO Hi: 5.6V UVLO Lo: 5.18V See Datasheet pg 15 Eq. 2+3 For calculating R3/R4"
- note removed: "brightness (PWM 0 - 255)"
