File: HW/HA_FONA_nonKiCad/HA_FONA_LARA_20.kicad_pcb (KiCad board)
At the start: 2 copper layers, 244.9 x 52.5 mm, 7 parts, among them X2 332-06

Commit message: Progress on HW .sch and .brd, with good portion of peripheral board finished, BQ25185 section incomplete and rocker switch section incomplete
Parts:
- removed X2: 332-06, HA_FONA_LARA_20-import-fps:332-06
- added C1: C_Polarized, Capacitor_THT:CP_Radial_D8.0mm_P5.00mm, F.Cu at (30.1, 63.8)
- added C2: 2.2u, Capacitor_SMD:C_0402_1005Metric, F.Cu at (48.3, 61.1)
- added C3: 0.1u, Capacitor_SMD:C_0402_1005Metric, F.Cu at (48.3, 63.0)
- added C4: 10u, Capacitor_SMD:C_0402_1005Metric, F.Cu at (48.3, 65.0)
- added C5: 1u, Capacitor_SMD:C_0402_1005Metric, F.Cu at (48.3, 67.0)
- added D2: D, Diode_THT:D_DO-15_P10.16mm_Horizontal, F.Cu at (30.2, 56.0)
- added J1: Conn_01x03_Pin, Connector_PinHeader_2.54mm:PinHeader_1x03_P2.54mm_Vertical, F.Cu at (27.5, 27.3)
- added J2: Conn_01x03_Pin, Connector_PinHeader_2.54mm:PinHeader_1x03_P2.54mm_Vertical, F.Cu at (48.1, 27.3)
- added Q1: PMOS, Package_TO_SOT_SMD:SOT-23, F.Cu at (40.7, 27.6)
- added U1: BQ25185DLHR, BQ25185DLHR:IC_BQ25185DLHR, F.Cu at (45.5, 71.4)
Routing:
- net Net-(D7-A): track 23.0 -> 38.6 mm
- net Net-(J2-Pin_3): track 0.00 -> 10.8 mm
- net Net-(J2-Pin_1): track 0.00 -> 8.90 mm
- net Net-(J2-Pin_2): track 0.00 -> 7.80 mm
- net Net-(D1-A): track 11.2 -> 18.1 mm
- net VBAT: track 24.0 -> 28.0 mm
- net Net-(D11-A): track 25.9 -> 29.5 mm
- net GND: track 29.2 -> 31.9 mm
