File: HW/HA_FONA_nonKiCad/HA_FONA_LARA_20.kicad_sch (KiCad schematic)
At the start: 7 parts, among them X2 332-06

Commit message: Progress on HW .sch and .brd, with good portion of peripheral board finished, BQ25185 section incomplete and rocker switch section incomplete
Parts:
- removed X2: 332-06, HA_FONA_LARA_20-import-fps:332-06, symbol HA_FONA_LARA_20-eagle-import:332-06
- added C1: C_Polarized, CP_Radial_D8.0mm_P5.00mm, symbol Device:C_Polarized
- added C2: 2.2u, Capacitor_SMD:C_0402_1005Metric, symbol Device:C
- added C3: 0.1u, Capacitor_SMD:C_0402_1005Metric, symbol Device:C
- added C4: 10u, Capacitor_SMD:C_0402_1005Metric, symbol Device:C
- added C5: 1u, Capacitor_SMD:C_0402_1005Metric, symbol Device:C
- added D2: D, D_DO-15_P10.16mm_Horizontal, symbol Device:D
- added J1, J2: Conn_01x03_Pin, Connector_PinHeader_2.54mm:PinHeader_1x03_P2.54mm_Vertical, symbol Connector:Conn_01x03_Pin
- added Q1: PMOS, Package_TO_SOT_SMD:SOT-23, symbol Simulation_SPICE:PMOS
- added U1: BQ25185DLHR, BQ25185DLHR:IC_BQ25185DLHR, symbol BQ25185D:BQ25185DLHR
- D11: footprint HA_FONA_LARA_20-import-fps:DIOM5336X265N -> Diode_SMD:D_SOD-123
Connections:
- net GND: now also C1.2, C2.1, C3.1, C4.2, C5.1, D2.2 (A), U1.5 (GND)
- net VBAT: now also C1.1, C2.2, C3.2, D2.1 (K), U1.10 (IN)
- net at D11.2 (A), D12.1 (C): now also J1.3 (Pin_3)
- net at D1.2 (A), D3.1 (C): now also J1.1 (Pin_1)
- net at D7.2 (A), D9.1 (C): now also J1.2 (Pin_2)
- new net: C5.2, U1.2 (BAT)
- new net: J2.3 (Pin_3), Q1.1 (D)
- new net: J2.2 (Pin_2), Q1.2 (G)
- new net: J2.1 (Pin_1), Q1.3 (S)
- new net: C4.1, U1.1 (SYS)
Other:
- note removed: "POWER AND FILTERING"
